File: V-00757-01.sch (EAGLE design)
At the start: 21 parts, among them IC1 MEGA8-AI, IC2 MAX481CSA, Q1 14.7456MHz

Commit message: v.2.0
Parts:
- removed U$2: SM04B-SRSS-TB-SIDE-TYPE, LIC_ALL-00:SM04B-SRSS-TB-SIDE-TYPE
- added R6: 0R, #PaJa_31:R_1206
- IO2: value LF50CDT -> 78M05; device #PaJa_31:LF_CDT -> #PaJa_31:78M
- R4: value 10k -> 100R
Connections:
- net +24V_OUT renamed +24V_IN
- removed net EMITOR: U$2.1
- removed net KATODA: U$2.3
- removed net N$11: CAN1.7
- removed net N$13: CAN1.9
- removed net N$4: IC1.PC0(ADC0), R5.2
- removed net N$7: CAN1.3
- new net N.C.0: CAN1.2
- new net N.C.1: CAN1.6
- new net N.C.2: CAN1.8
- net +5V: now also CAN1.7; no longer CAN1.4
- net ANODA: no longer U$2.4
- net BUS_A: now also CAN1.9; no longer CAN1.6
- net BUS_B: now also CAN1.3; no longer CAN1.8
- net GND: now also CAN1.4; no longer CAN1.2, U$2.GND0, U$2.GND1
- net KOLEKTOR: now also IC1.PC0(ADC0), R5.2; no longer U$2.2
Other:
- note added: "Nas novy standard s napajenim!!! Dle standardu je 1. +24 V 2. RXD+ 3. Data+ (B) 4. GND 5. GND 6. RXD- 7. +5 V 8. Nevyuzit 9. Data- (A)"
Changed lines of the file:
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@@
 <part name="CAN1" library="#PaJa_konektory" deviceset="CAN_9V" device="_/90" value="CAN_9V_/90"/>
 <part name="D1" library="diode" deviceset="MBRS3*0T3" device="" technology="4"/>
-<part name="IO2" library="#PaJa_31" deviceset="LF_C" device="DT" value="LF50CDT"/>
+<part name="IO2" library="#PaJa_31" deviceset="78?" device="M" value="78M05"/>
 <part name="C5" library="#PaJa_31" deviceset="C-KER" device="_1206" value="10uF"/>
 <part name="C6" library="#PaJa_31" deviceset="C-KER" device="_1206" value="100n"/>
 <part name="U$1" library="#PaJa_konektory" deviceset="AVR_PROG_SPI" device=""/>
-<part name="U$2" library="LIC_ALL-00" deviceset="SM04B-SRSS-TB" device="-SIDE-TYPE"/>
 <part name="K1" library="#PaJa_konektory" deviceset="PSH02-04" device="W"/>
-<part name="R4" library="#PaJa_31" deviceset="R" device="_1206" value="10k"/>
+<part name="R4" library="#PaJa_31" deviceset="R" device="_1206" value="100R"/>
 <part name="R5" library="#PaJa_31" deviceset="R" device="_1206" value="1k"/>
+<part name="R6" library="#PaJa_31" deviceset="R" device="_1206" value="0R"/>
 </parts>
 <sheets>
@@
 3. Katoda
 4. Anoda</text>
+<text x="200.66" y="119.38" size="1.778" layer="97" align="top-left">Nas novy standard s napajenim!!!
+Dle standardu je
+1. +24 V
+2. RXD+
+3. Data+ (B)
+4. GND
+5. GND
+6. RXD-
+7. +5 V
+8. Nevyuzit
+9. Data- (A)</text>
 </plain>
 <instances>
@@
 <instance part="C6" gate="C" x="139.7" y="162.56" rot="R90"/>
 <instance part="U$1" gate="G$1" x="182.88" y="63.5" rot="R270"/>
-<instance part="U$2" gate="G$1" x="231.14" y="109.22"/>
 <instance part="K1" gate="KON" x="205.74" y="144.78" rot="R270"/>
 <instance part="R4" gate="R" x="124.46" y="129.54"/>
 <instance part="R5" gate="R" x="119.38" y="144.78" rot="R270"/>
+<instance part="R6" gate="R" x="111.76" y="63.5" rot="R180"/>
 </instances>
 <busses>
@@
 </segment>
 <segment>
-<pinref part="CAN1" gate="CAN" pin="6"/>
-<wire x1="210.82" y1="63.5" x2="210.82" y2="55.88" width="0.1524" layer="91"/>
-<label x="210.82" y="55.88" size="1.016" layer="95" font="vector" ratio="10" rot="R270" xref="yes"/>
+<pinref part="CAN1" gate="CAN" pin="9"/>
+<wire x1="226.06" y1="63.5" x2="226.06" y2="55.88" width="0.1524" layer="91"/>
+<label x="226.06" y="55.88" size="1.016" layer="95" font="vector" ratio="10" rot="R270" xref="yes"/>
 </segment>
 </net>
@@
 </segment>
 <segment>
-<pinref part="CAN1" gate="CAN" pin="8"/>
-<wire x1="220.98" y1="63.5" x2="220.98" y2="55.88" width="0.1524" layer="91"/>
-<label x="220.98" y="55.88" size="1.016" layer="95" font="vector" ratio="10" rot="R270" xref="yes"/>
+<pinref part="CAN1" gate="CAN" pin="3"/>
+<wire x1="218.44" y1="68.58" x2="218.44" y2="76.2" width="0.1524" layer="91"/>
+<label x="218.44" y="76.2" size="1.016" layer="95" font="vector" ratio="10" rot="R90" xref="yes"/>
 </segment>
 </net>
@@
 </segment>
 <segment>
-<pinref part="CAN1" gate="CAN" pin="4"/>
-<wire x1="223.52" y1="68.58" x2="223.52" y2="76.2" width="0.1524" layer="91"/>
-<label x="223.52" y="76.2" size="1.016" layer="95" font="vector" ratio="10" rot="R90" xref="yes"/>
-</segment>
-<segment>
 <pinref part="R5" gate="R" pin="1"/>
 <wire x1="119.38" y1="149.86" x2="119.38" y2="152.4" width="0.1524" layer="91"/>
 <wire x1="119.38" y1="152.4" x2="116.84" y2="152.4" width="0.1524" layer="91"/>
 <label x="116.84" y="152.4" size="1.27" layer="95" font="vector" ratio="10" rot="R180" xref="yes"/>
+</segment>
+<segment>
+<pinref part="CAN1" gate="CAN" pin="7"/>
+<wire x1="215.9" y1="63.5" x2="215.9" y2="55.88" width="0.1524" layer="91"/>
+<label x="215.9" y="55.88" size="1.016" layer="95" font="vector" ratio="10" rot="R270" xref="yes"/>
 </segment>
 </net>
@@
 </segment>
 <segment>
-<pinref part="CAN1" gate="CAN" pin="2"/>
-<wire x1="213.36" y1="68.58" x2="213.36" y2="76.2" width="0.1524" layer="91"/>
-<label x="213.36" y="76.2" size="1.016" layer="95" font="vector" ratio="10" rot="R90" xref="yes"/>
-</segment>
-<segment>
-<pinref part="U$2" gate="G$1" pin="GND0"/>
-<wire x1="238.76" y1="119.38" x2="238.76" y2="121.92" width="0.1524" layer="91"/>
-<wire x1="238.76" y1="121.92" x2="226.06" y2="121.92" width="0.1524" layer="91"/>
-<label x="226.06" y="121.92" size="1.016" layer="95" font="vector" ratio="12" rot="R180" xref="yes"/>
-</segment>
-<segment>
-<pinref part="U$2" gate="G$1" pin="GND1"/>
-<wire x1="238.76" y1="96.52" x2="238.76" y2="93.98" width="0.1524" layer="91"/>
-<wire x1="238.76" y1="93.98" x2="226.06" y2="93.98" width="0.1524" layer="91"/>
-<label x="226.06" y="93.98" size="1.016" layer="95" font="vector" ratio="12" rot="R180" xref="yes"/>
-</segment>
-<segment>
 <pinref part="K1" gate="KON" pin="3"/>
 <wire x1="203.2" y1="142.24" x2="195.58" y2="142.24" width="0.1524" layer="91"/>
@@
 <wire x1="203.2" y1="147.32" x2="195.58" y2="147.32" width="0.1524" layer="91"/>
 <label x="195.58" y="147.32" size="1.016" layer="95" font="vector" ratio="10" rot="R180" xref="yes"/>
+</segment>
+<segment>
+<pinref part="CAN1" gate="CAN" pin="4"/>
+<wire x1="223.52" y1="68.58" x2="223.52" y2="76.2" width="0.1524" layer="91"/>
+<label x="223.52" y="76.2" size="1.016" layer="95" font="vector" ratio="10" rot="R90" xref="yes"/>
 </segment>
 </net>
@@
 </segment>
 </net>
-<net name="N$7" class="0">
-<segment>
-<pinref part="CAN1" gate="CAN" pin="3"/>
-<wire x1="218.44" y1="68.58" x2="218.44" y2="76.2" width="0.1524" layer="91"/>
-<label x="218.44" y="76.2" size="1.016" layer="95" font="vector" ratio="10" rot="R90" xref="yes"/>
-</segment>
-</net>
-<net name="N$11" class="0">
-<segment>
-<pinref part="CAN1" gate="CAN" pin="7"/>
-<wire x1="215.9" y1="63.5" x2="215.9" y2="55.88" width="0.1524" layer="91"/>
-<label x="215.9" y="55.88" size="1.016" layer="95" font="vector" ratio="10" rot="R270" xref="yes"/>
-</segment>
-</net>
-<net name="N$13" class="0">
-<segment>
-<pinref part="CAN1" gate="CAN" pin="9"/>
-<wire x1="226.06" y1="63.5" x2="226.06" y2="55.88" width="0.1524" layer="91"/>
-<label x="226.06" y="55.88" size="1.016" layer="95" font="vector" ratio="10" rot="R270" xref="yes"/>
-</segment>
-</net>
-<net name="+24V_OUT" class="0">
+<net name="+24V_IN" class="0">
 <segment>
 <pinref part="D1" gate="G$1" pin="A"/>
@@
 <net name="ANODA" class="0">
 <segment>
-<pinref part="U$2" gate="G$1" pin="4"/>
-<wire x1="226.06" y1="111.76" x2="213.36" y2="111.76" width="0.1524" layer="91"/>
-<label x="213.36" y="111.76" size="1.016" layer="95" font="vector" ratio="12" rot="R180" xref="yes"/>
-</segment>
-<segment>
 <pinref part="K1" gate="KON" pin="4"/>
 <wire x1="203.2" y1="139.7" x2="195.58" y2="139.7" width="0.1524" layer="91"/>
@@
 </segment>
 </net>
-<net name="KATODA" class="0">
-<segment>
-<pinref part="U$2" gate="G$1" pin="3"/>
-<wire x1="226.06" y1="109.22" x2="213.36" y2="109.22" width="0.1524" layer="91"/>
-<label x="213.36" y="109.22" size="1.016" layer="95" font="vector" ratio="12" rot="R180" xref="yes"/>
-</segment>
-</net>
 <net name="KOLEKTOR" class="0">
-<segment>
-<pinref part="U$2" gate="G$1" pin="2"/>
-<wire x1="226.06" y1="106.68" x2="213.36" y2="106.68" width="0.1524" layer="91"/>
-<label x="213.36" y="106.68" size="1.016" layer="95" font="vector" ratio="12" rot="R180" xref="yes"/>
-</segment>
 <segment>
 <pinref part="K1" gate="KON" pin="2"/>
@@
 <label x="195.58" y="144.78" size="1.016" layer="95" font="vector" ratio="10" rot="R180" xref="yes"/>
 </segment>
-</net>
-<net name="EMITOR" class="0">
-<segment>
-<pinref part="U$2" gate="G$1" pin="1"/>
-<wire x1="226.06" y1="104.14" x2="213.36" y2="104.14" width="0.1524" layer="91"/>
-<label x="213.36" y="104.14" size="1.016" layer="95" font="vector" ratio="12" rot="R180" xref="yes"/>
-</segment>
-</net>
-<net name="N$3" class="0">
-<segment>
-<pinref part="IC1" gate="G$1" pin="PC3(ADC3)"/>
-<pinref part="R4" gate="R" pin="1"/>
-<wire x1="114.3" y1="129.54" x2="119.38" y2="129.54" width="0.1524" layer="91"/>
-</segment>
-</net>
-<net name="N$4" class="0">
 <segment>
 <pinref part="IC1" gate="G$1" pin="PC0(ADC0)"/>
@@
 <wire x1="119.38" y1="137.16" x2="124.46" y2="137.16" width="0.1524" layer="91"/>
 <junction x="119.38" y="137.16"/>
-</segment>
-</net>
+<label x="124.46" y="137.16" size="1.016" layer="95" ratio="10" xref="yes"/>
+</segment>
+</net>
+<net name="N$3" class="0">
+<segment>
+<pinref part="IC1" gate="G$1" pin="PC3(ADC3)"/>
+<pinref part="R4" gate="R" pin="1"/>
+<wire x1="114.3" y1="129.54" x2="119.38" y2="129.54" width="0.1524" layer="91"/>
+</segment>
+</net>
+<net name="N.C.0" class="0">
+<segment>
+<pinref part="CAN1" gate="CAN" pin="2"/>
+<wire x1="213.36" y1="68.58" x2="213.36" y2="76.2" width="0.1524" layer="91"/>
+<label x="213.36" y="76.2" size="1.016" layer="95" font="vector" ratio="10" rot="R90" xref="yes"/>
+</segment>
+</net>
+<net name="N.C.1" class="0">
+<segment>
+<pinref part="CAN1" gate="CAN" pin="6"/>
+<wire x1="210.82" y1="63.5" x2="210.82" y2="55.88" width="0.1524" layer="91"/>
+<label x="210.82" y="55.88" size="1.016" layer="95" font="vector" ratio="10" rot="R270" xref="yes"/>
+</segment>
+</net>
+<net name="N.C.2" class="0">
+<segment>
+<pinref part="CAN1" gate="CAN" pin="8"/>
+<wire x1="220.98" y1="63.5" x2="220.98" y2="55.88" width="0.1524" layer="91"/>
+<label x="220.98" y="55.88" size="1.016" layer="95" font="vector" ratio="10" rot="R270" xref="yes"/>
+</segment>
+</net>
